Commit message: Fixed some issues with r2000ib100p

File: fanuc_r2000ib_support/urdf/r2000ib.ros2_control.xacro (robot description, xacro)
@@ -12,5 +12,5 @@
         <!-- physical hardware or RobotStudio simulation -->
         <xacro:unless value="${use_fake_hardware}">
-          <plugin>abb_hardware_interface/ABBSystemHardware</plugin>
+          <!-- <plugin>abb_hardware_interface/ABBSystemHardware</plugin> -->
           <!-- If false, the robot description required for EGM connection-->
           <!-- will be generated as per joint information listed below. -->

File: fanuc_r2000ib_support/urdf/r2000ib100p_macro.xacro (robot description, xacro)
@@ -210,5 +210,5 @@
     <link name="${prefix}flange"/>
     <joint type="fixed" name="${prefix}joint_6-flange">
-      <origin xyz="0 0 0" rpy="0 0 0"/>
+      <origin xyz="0 0 0" rpy="0 -${radians(90)} 0"/>
       <parent link="${prefix}link_6"/>
       <child link="${prefix}flange"/>
@@ -217,6 +217,6 @@
     <link name="${prefix}tool0" />
     <joint name="${prefix}link_6-tool0" type="fixed">
-      <origin xyz="0 0 0" rpy="0 ${radians(90)} 0" />
-      <parent link="${prefix}flange" />
+      <origin xyz="0 0 0" rpy="0 0 -${radians(180)}" />
+      <parent link="${prefix}link_6" />
       <child link="${prefix}tool0" />
     </joint>
